Commit message: submodules

File: summit_xl_description/robots/summit_xls_std.urdf.xacro (robot description, xacro)
@@ -65,12 +65,12 @@
 		</xacro:omni_wheel>
         <!-- IMU -->
-		<xacro:sensor_imu prefix="$(arg prefix)imu" parent="$(arg prefix)base_link">
+		<xacro:sensor_imu prefix="$(arg prefix)imu" parent="$(arg prefix)base_link" sensor_name="IMU">
 			<origin xyz="${imu_offset_x} ${imu_offset_y} ${imu_offset_z}" rpy="0 0 0"/>
 		</xacro:sensor_imu>
 		<!-- SENSORS -->
-		<xacro:sensor_sick_s300 prefix="$(arg prefix)front_laser" parent="$(arg prefix)base_link" prefix_topic="front_laser" gpu="$(arg gpu)">
+		<xacro:sensor_sick_s300 prefix="$(arg prefix)front_laser" parent="$(arg prefix)base_link" prefix_topic="front_laser" gpu="$(arg gpu)" sensor_name="FLIDAR">
 			<origin xyz="${front_laser_offset_x} ${front_laser_offset_y} ${front_laser_offset_z}" rpy="0 ${-PI} ${3/4*PI}" />
 		</xacro:sensor_sick_s300>
-		<xacro:sensor_sick_s300 prefix="$(arg prefix)rear_laser" parent="$(arg prefix)base_link" prefix_topic="rear_laser" gpu="$(arg gpu)">
+		<xacro:sensor_sick_s300 prefix="$(arg prefix)rear_laser" parent="$(arg prefix)base_link" prefix_topic="rear_laser" gpu="$(arg gpu)" sensor_name="BLIDAR">
 			<origin xyz="${rear_laser_offset_x} ${rear_laser_offset_y} ${rear_laser_offset_z}" rpy="0 ${-PI} ${-1/4*PI}" />
 		</xacro:sensor_sick_s300>
@@ -93,3 +93,17 @@
    </xacro:if>
    <xacro:summit_xl prefix="$(arg prefix)" publish_bf="true" hq="true"/>
+ <gazebo reference="$(arg prefix)base_link">
+   <sensor name='body_contact' type='contact'>
+          <contact>
+            <!--<collision>robot::robot_base_footprint::robot_base_footprint_fixed_joint_lump__robot_base_link_collision</collision>-->
+<collision>robot_base_footprint_fixed_joint_lump__robot_base_link_collision</collision>
+<topic>__default_topic__</topic>
+          </contact>
+   <plugin name="body_plugin" filename="libgazebo_ros_bumper.so">
+     	<alwaysOn>true</alwaysOn>
+         <bumperTopicName>body_contact</bumperTopicName>
+         <frameName>$(arg prefix)base_footprint</frameName>
+   </plugin>
+   </sensor>
+  </gazebo>
 </robot>

File: summit_xl_description/urdf/bases/summit_xls_base.urdf.xacro (robot description, xacro)
@@ -22,4 +22,22 @@
 		</joint>
 	  </xacro:if>
+<!-- COLLISON
+  <link name="${prefix}collision_box">
+  <origin xyz="0 0 0" rpy="0 0 0" />
+  <geometry>
+	 <box size="0.8 0.8 0.8" />
+  </geometry>
+    <collision name="${prefix}collision_box">
+      <geometry>
+        <box size="0.8 0.8 0.8" />
+      </geometry>
+    </collision>
+  </link>
+  <joint name="box_joint" type="fixed">
+    <parent link="${prefix}base_link"/>
+    <child link="${prefix}collision_box"/>
+    <origin xyz="0.0 0.0 0.5" rpy="0 0 0"/>
+  </joint>
+-->
   <!-- BASE_LINK -->
   <link name="${prefix}base_link">

Commit message: added contact sensor

File: summit_xl_description/robots/summit_xls_std.urdf.xacro (robot description, xacro)
@@ -93,3 +93,16 @@
    </xacro:if>
    <xacro:summit_xl prefix="$(arg prefix)" publish_bf="true" hq="true"/>
+   <gazebo reference="robot_base_footprint">
+   <sensor name='body_contact' type='contact'>
+          <contact>
+            <collision>robot_base_footprint_fixed_joint_lump__robot_base_link_collision</collision>
+	   <topic>__default_topic__</topic>
+          </contact>
+   <plugin name="body_plugin" filename="libgazebo_ros_bumper.so">
+     	<alwaysOn>true</alwaysOn>
+         <bumperTopicName>body_contact</bumperTopicName>
+         <frameName>robot_base_footprint</frameName>
+   </plugin>
+   </sensor>
+   </gazebo>
 </robot>
